Commit message: navigation launch file added

File: hanwhabot_description/urdf/hanwhabot_v1.urdf.xacro (robot description, xacro)
@@ -12,14 +12,8 @@
       <geometry>
         <!-- plz input right value -->
-        <box size="0.140 0.140 0.30"/>
+        <box size="0.680 0.465 0.30"/>
       </geometry>
       <material name="light_black"/>
     </visual>
-    <collision>
-      <origin xyz="-0.032 0 0.070" rpy="0 0 0"/>
-      <geometry>
-        <box size="0.140 0.140 0.143"/>
-      </geometry>
-    </collision>
   </link>
   <joint name="wheel_left_joint" type="continuous">

Commit message: navigation commit

File: hanwhabot_description/urdf/hanwhabot_v1.urdf.xacro (robot description, xacro)
@@ -5,9 +5,9 @@
     <parent link="base_footprint"/>
     <child link="base_link"/>
-    <origin xyz="0.0 0.0 0.010" rpy="0 0 0"/>
+    <origin xyz="0.0 0.0 0.01" rpy="0 0 0"/>
   </joint>
   <link name="base_link">
     <visual>
-      <origin xyz="-0.032 0 0.0" rpy="0 0 0"/>
+      <origin xyz="0 0 0" rpy="0 0 0"/>
       <geometry>
         <!-- plz input right value -->
@@ -17,52 +17,52 @@
     </visual>
   </link>
-  <joint name="wheel_left_joint" type="continuous">
+  <!-- <joint name="wheel_left_joint" type="continuous">
     <parent link="base_link"/>
     <child link="wheel_left_link"/>
-    <origin xyz="0.0 0.08 0.023" rpy="-1.57 0 0"/>
+    <origin xyz="0.0 0.233 0.0" rpy="-1.57 0 0"/>
     <axis xyz="0 0 1"/>
-  </joint>
-  <link name="wheel_left_link">
-    <visual>
+  </joint> -->
+  <!-- <link name="wheel_left_link"> -->
+    <!-- <visual>
       <origin xyz="0 0 0" rpy="1.57 0 0"/>
       <geometry>
-        <!-- <mesh filename="package://turtlebot3_description/meshes/wheels/left_tire.stl" scale="0.001 0.001 0.001"/> -->
+          <cylinder length="0.088" radius="0.0475"/>
       </geometry>
       <material name="dark"/>
-    </visual>
-    <collision>
+    </visual> -->
+    <!-- <collision>
       <origin xyz="0 0 0" rpy="0 0 0"/>
       <geometry>
         <cylinder length="0.018" radius="0.033"/>
       </geometry>
-    </collision>
-  </link>
-  <joint name="wheel_right_joint" type="continuous">
+    </collision> -->
+  <!-- </link> -->
+  <!-- <joint name="wheel_right_joint" type="continuous">
     <parent link="base_link"/>
     <child link="wheel_right_link"/>
-    <origin xyz="0.0 -0.080 0.023" rpy="-1.57 0 0"/>
+    <origin xyz="0.0 -0.233 0.0" rpy="-1.57 0 0"/>
     <axis xyz="0 0 1"/>
-  </joint>
-  <link name="wheel_right_link">
-    <visual>
+  </joint> -->
+  <!-- <link name="wheel_right_link"> -->
+    <!-- <visual>
       <origin xyz="0 0 0" rpy="1.57 0 0"/>
       <geometry>
-        <!-- <mesh filename="package://turtlebot3_description/meshes/wheels/right_tire.stl" scale="0.001 0.001 0.001"/> -->
+        <cylinder length="0.088" radius="0.0475"/>
       </geometry>
       <material name="dark"/>
-    </visual>
-    <collision>
+    </visual> -->
+    <!-- <collision>
       <origin xyz="0 0 0" rpy="0 0 0"/>
       <geometry>
         <cylinder length="0.018" radius="0.033"/>
       </geometry>
-    </collision>
-  </link>
-  <joint name="caster_back_joint" type="fixed">
+    </collision> -->
+  <!-- </link> -->
+  <!-- <joint name="caster_back_joint" type="fixed">
     <parent link="base_link"/>
     <child link="caster_back_link"/>
     <origin xyz="-0.081 0 -0.004" rpy="-1.57 0 0"/>
-  </joint>
-  <link name="caster_back_link">
+  </joint> -->
+  <!-- <link name="caster_back_link">
     <collision>
       <origin xyz="0 0.001 0" rpy="0 0 0"/>
@@ -72,29 +72,24 @@
     </collision>
   </link>
+ -->
   <link name="imu_link"/>
   <joint name="imu_joint" type="fixed">
     <parent link="base_link"/>
     <child link="imu_link"/>
-    <origin xyz="-0.032 0 0.068" rpy="0 0 0"/>
+    <origin xyz="-0.32 0 0.15" rpy="0 0 0"/>
   </joint>
   <joint name="scan_joint" type="fixed">
     <parent link="base_link"/>
     <child link="base_scan"/>
-    <origin xyz="-0.032 0 0.172" rpy="0 0 0"/>
+    <origin xyz="0.34 0 0.14" rpy="0 0 0"/>
   </joint>
   <link name="base_scan">
     <visual>
-      <origin xyz="0 0 0.0" rpy="0 0 0"/>
+      <origin xyz="0.34 0 0.14" rpy="0 0 0"/>
       <geometry>
-        <!-- <mesh filename="package://turtlebot3_description/meshes/sensors/lds.stl" scale="0.001 0.001 0.001"/> -->
+        <cylinder length="0.088" radius="0.0475"/>
       </geometry>
-      <material name="dark"/>
+      <material name="white"/>
     </visual>
-    <collision>
-      <origin xyz="0.015 0 -0.0065" rpy="0 0 0"/>
-      <geometry>
-        <cylinder length="0.0315" radius="0.055"/>
-      </geometry>
-    </collision>
   </link>
   <link name="camera_link"/>
@@ -102,5 +97,5 @@
     <parent link="base_link"/>
     <child link="camera_link"/>
-    <origin xyz="-0.032 0 0.068" rpy="0 0 0"/>
+    <origin xyz="0.34 0 0.15" rpy="0 0 0"/>
   </joint>
 </robot>
